File: hardware/button-grid.kicad_sch (KiCad schematic)
At the start: 68 parts, among them J1 12V DC, J2 USB-C, J3 ROWS, J4 COLS, J5 UART, SW1 RESET, SW2 BOOT, U1 ESP32-S3-WROOM-1-N8, U2 TPS54202H

Commit message: Fully routed board: 0 DRC errors, ERC/netlist checks pass
- autorouted with Freerouting (10um clearance margin), locked USB VBUS bridge
- GND pours both sides, stitching vias, solid GND on THT pins
- run checks on every branch; Pages deploy from main

Co-Authored-By: Claude Opus 5.5 <noreply@anthropic.com>
Claude-Session: https://claude.ai/code/session_01USgdVYHDQPVjqMcbCmVwPa
Parts:
- H1, H2, H3, H4: now left out of the parts list
Changed lines of the file:
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@@
 		(unit 1)
 		(exclude_from_sim no)
-		(in_bom yes)
+		(in_bom no)
 		(on_board yes)
 		(dnp no)
@@
 		(unit 1)
 		(exclude_from_sim no)
-		(in_bom yes)
+		(in_bom no)
 		(on_board yes)
 		(dnp no)
@@
 		(unit 1)
 		(exclude_from_sim no)
-		(in_bom yes)
+		(in_bom no)
 		(on_board yes)
 		(dnp no)
@@
 		(unit 1)
 		(exclude_from_sim no)
-		(in_bom yes)
-		(on_board yes)
-		(dnp no)
+		(in_bom no)
+		(on_board yes)
+		(dnp no)
